Commit message: urdf file

File: urdf/tnbd_proto5.urdf (robot description, URDF)
Before this commit: robot tnbd_proto5, 9 links, 8 joints
Joints:
- joint back_joint: limit lower=0 upper=0 effort=0 velocity=0 -> lower=-1.570796 upper=0 effort=0 velocity=0
- joint feed_joint: limit lower=0 upper=0 effort=0 velocity=0 -> lower=-0.802851 upper=0 effort=0 velocity=0
- joint front_joint: limit lower=0 upper=0 effort=0 velocity=0 -> lower=0 upper=2.000321 effort=0 velocity=0

Commit message: twice commit

File: urdf/tnbd_proto5.urdf (robot description, URDF)
Before this commit: robot tnbd_proto5, 9 links, 8 joints
Links:
- removed link left_wheel_link
- removed link lidar_link
- removed link opencr_link
- removed link right_wheel_link
- added link base_footprint
- added link base_scan, mass 0.131767415545665; collision mesh filename=package://tnbd_proto5/meshes/lidar_link.STL; visual mesh filename=package://tnbd_proto5/meshes/lidar_link.STL
- added link imu_link, mass 5.58945396958244; collision mesh filename=package://tnbd_proto5/meshes/opencr_link.STL; visual mesh filename=package://tnbd_proto5/meshes/opencr_link.STL
- added link wheel_left_link, mass 0.431849530870227; collision mesh filename=package://tnbd_proto5/meshes/left_wheel_link.STL; visual mesh filename=package://tnbd_proto5/meshes/left_wheel_link.STL
- added link wheel_right_link, mass 0.431849530870227; collision mesh filename=package://tnbd_proto5/meshes/right_wheel_link.STL; visual mesh filename=package://tnbd_proto5/meshes/right_wheel_link.STL
Joints:
- removed joint left_wheel_joint
- removed joint lidar_joint
- removed joint opencr_joint
- removed joint right_wheel_joint
- added joint base_joint: type fixed, parent base_footprint, child base_link, origin xyz=-0.0132838481327496 -0.0190930870578007 -0.0165104491009677 rpy=0 0 0
- added joint imu_joint: type fixed, parent base_link, child imu_link, origin xyz=0 0 0 rpy=0 0 -3.1416, axis 0 0 0
- added joint scan_joint: type fixed, parent base_link, child base_scan, origin xyz=-0.035043 0.0083315 0.077 rpy=0 0 0, axis 0 0 0
- added joint wheel_left_joint: type continuous, parent base_link, child wheel_left_link, origin xyz=0.027457 -0.12147 -0.0339 rpy=-1.5708 0.62286 -3.1416, axis 0 0 1
- added joint wheel_right_joint: type continuous, parent base_link, child wheel_right_link, origin xyz=0.027457 0.13813 -0.0339 rpy=1.5708 -0.0072638 0, axis 0 0 1
- joint front_joint: origin xyz=-0.15554 0 -0.06 rpy=2.7278 0 -1.5708 -> xyz=-0.15554 0 0 rpy=2.7278 0 -1.5708
